File: kicad/MegaGRRLDesktop.kicad_pcb (KiCad board)
At the start: 2 copper layers, 124.5 x 124.5 mm, 133 parts, among them IC10 PCA9634PW, IC11 TPA6111A2DR, IC12 ESP-WROOM-32ESP-WROOM-32-NO-RF, IC14 CH340C, IC2 74HCT595N, IC3 74HCT595N, IC4 MCP23017SP, IC5 NE5532N, IC6 std:a4c6558b222b489b868198a35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, IC6A std:44d60e1deb274ae4bbd12617d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

Commit message: 0.47
Parts:
- moved G*** 3.08 mm to (148.8, 99.0)
- moved G*** 1.30 mm to (145.6, 161.4)
- moved G*** 0.80 mm to (148.6, 66.6)
Changed lines of the file:
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@@
   )
   (footprint "Silk Screen Art:MegaGRRL Desktop" (layer "F.Cu")
-    (at 146.422721 162.403457)
+    (at 145.6 161.4)
     (attr board_only exclude_from_pos_files exclude_from_bom)
     (fp_text reference "G***" (at -2.922721 10.896543) (layer "F.SilkS")
@@
   )
   (footprint "Silk Screen Art:heart on fire" (layer "B.Cu")
-    (at 149.4 66.6 180)
+    (at 148.6 66.6 180)
     (attr board_only exclude_from_pos_files exclude_from_bom)
     (fp_text reference "G***" (at 0 0) (layer "B.SilkS") hide
@@
   )
   (footprint "Silk Screen Art:natalie-md" (layer "B.Cu")
-    (at 146.069765 97.581607 180)
+    (at 148.8 99 180)
     (attr board_only exclude_from_pos_files exclude_from_bom)
     (fp_text reference "G***" (at 0 0) (layer "B.SilkS") hide
