File: kicad/MegaGRRLDesktop.kicad_pcb-v0.47.kicad_pcb (KiCad board)
At the start: 2 copper layers, 124.5 x 124.5 mm, 133 parts, among them IC10 PCA9634PW, IC11 TPA6111A2DR, IC12 ESP-WROOM-32ESP-WROOM-32-NO-RF, IC14 CH340C, IC2 74HCT595N, IC3 74HCT595N, IC4 MCP23017SP, IC5 NE5532N, IC6 std:a4c6558b222b489b868198a35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, IC6A std:44d60e1deb274ae4bbd12617d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

Commit message: 2024.7.7
Changed lines of the file:
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@@
     (property "Sheetfile" "LED_drivers.kicad_sch")
     (property "Sheetname" "LED drivers")
-    (fp_text reference "RN3" (at 11.43 0) (layer "F.SilkS")
+    (fp_text reference "RN3" (at 15.24 -0.635) (layer "F.SilkS")
         (effects (font (size 1.1557 1.1557) (thickness 0.1143)) (justify right))
     )
@@
         (effects (font (size 1.1557 1.1557) (thickness 0.1143)) (justify right))
     )
-    (fp_text user "1" (at -11.43 -0.508 180) (layer "F.SilkS")
+    (fp_text user "1" (at -12.446 0.508 180) (layer "F.SilkS")
         (effects (font (size 0.871728 0.871728) (thickness 0.118872)) (justify left bottom))
     )
@@
     (property "Sheetfile" "LED_drivers.kicad_sch")
     (property "Sheetname" "LED drivers")
-    (fp_text reference "RN1" (at 11.43 0) (layer "F.SilkS")
+    (fp_text reference "RN1" (at 15.24 -0.635) (layer "F.SilkS")
         (effects (font (size 1.1557 1.1557) (thickness 0.1143)) (justify right))
     )
@@
         (effects (font (size 1.1557 1.1557) (thickness 0.1143)) (justify right))
     )
-    (fp_text user "1" (at -11.43 -0.508 180) (layer "F.SilkS")
+    (fp_text user "1" (at -12.446 0.508 180) (layer "F.SilkS")
         (effects (font (size 0.871728 0.871728) (thickness 0.118872)) (justify left bottom))
     )
@@
   (segment (start 172.589 133.902724) (end 172.982676 134.2964) (width 0.25) (layer "F.Cu") (net 9))
   (segment (start 112.3061 105.6386) (end 119.5451 105.6386) (width 0.8128) (layer "F.Cu") (net 9))
-  (segment (start 117.4 101.2) (end 118.1 100.5) (width 0.8128) (layer "F.Cu") (net 9))
+  (segment (start 117.9 101.2) (end 118.3204 100.7796) (width 0.8128) (layer "F.Cu") (net 9))
   (segment (start 105.9561 102.4636) (end 102.1461 102.4636) (width 0.3048) (layer "F.Cu") (net 9))
   (segment (start 122.4661 79.6036) (end 120.5611 77.6986) (width 0.8128) (layer "F.Cu") (net 9))
   (segment (start 169.4561 134.2136) (end 171.6569 134.2136) (width 0.4064) (layer "F.Cu") (net 9))
-  (segment (start 117.3 101.2) (end 117.4 101.2) (width 0.8128) (layer "F.Cu") (net 9))
   (segment (start 124.1 79.6) (end 124.0964 79.6036) (width 0.8128) (layer "F.Cu") (net 9))
   (segment (start 118.1 87.5) (end 118.1 78.8897) (width 0.8128) (layer "F.Cu") (net 9))
+  (segment (start 117.3 101.2) (end 112.8614 105.6386) (width 0.8128) (layer "F.Cu") (net 9))
   (segment (start 124.0964 79.6036) (end 122.4661 79.6036) (width 0.8128) (layer "F.Cu") (net 9))
   (segment (start 119.2911 72.6186) (end 119.2911 77.6986) (width 0.8128) (layer "F.Cu") (net 9))
@@
   (segment (start 119.9261 106.2736) (end 129.7051 115.7986) (width 0.8128) (layer "F.Cu") (net 9))
   (segment (start 118.1 87.5) (end 117.405 86.805) (width 0.8128) (layer "F.Cu") (net 9))
-  (segment (start 112.3061 105.6386) (end 112.8614 105.6386) (width 0.8128) (layer "F.Cu") (net 9))
   (segment (start 145.9611 115.7986) (end 149.0561 112.7036) (width 0.8128) (layer "F.Cu") (net 9))
   (segment (start 102.1461 102.4636) (end 101.5111 103.0986) (width 0.3048) (layer "F.Cu") (net 9))
@@
   (segment (start 101.5111 103.0986) (end 101.5111 108.8136) (width 0.3048) (layer "F.Cu") (net 9))
   (segment (start 101.5111 108.8136) (end 102.1461 109.4486) (width 0.3048) (layer "F.Cu") (net 9))
-  (segment (start 118.1 100.5) (end 118.1 87.5) (width 0.8128) (layer "F.Cu") (net 9))
   (segment (start 171.6569 134.2136) (end 172.589 133.2815) (width 0.4064) (layer "F.Cu") (net 9))
   (segment (start 107.2261 104.2136) (end 107.2261 103.7336) (width 0.3048) (layer "F.Cu") (net 9))
@@
   (segment (start 117.405 86.805) (end 116.3 86.805) (width 0.8128) (layer "F.Cu") (net 9))
   (segment (start 124.1 79.6) (end 125.5 79.6) (width 0.8128) (layer "F.Cu") (net 9))
+  (segment (start 112.8614 105.6386) (end 112.3061 105.6386) (width 0.8128) (layer "F.Cu") (net 9))
   (segment (start 108.6511 105.6386) (end 107.2261 104.2136) (width 0.3048) (layer "F.Cu") (net 9))
   (segment (start 108.6511 105.6386) (end 112.3061 105.6386) (width 0.4064) (layer "F.Cu") (net 9))
-  (segment (start 112.8614 105.6386) (end 117.3 101.2) (width 0.8128) (layer "F.Cu") (net 9))
+  (segment (start 118.1 99.7) (end 118.1 87.5) (width 0.8128) (layer "F.Cu") (net 9))
   (segment (start 149.0561 112.7036) (end 156.1211 112.7036) (width 0.8128) (layer "F.Cu") (net 9))
   (segment (start 172.982676 134.2964) (end 174.145324 134.2964) (width 0.25) (layer "F.Cu") (net 9))
+  (segment (start 118.3204 99.9204) (end 118.1 99.7) (width 0.8128) (layer "F.Cu") (net 9))
+  (segment (start 117.9 101.2) (end 117.3 101.2) (width 0.8128) (layer "F.Cu") (net 9))
   (segment (start 116.105 87) (end 101 87) (width 0.8128) (layer "F.Cu") (net 9))
   (segment (start 120.5611 77.6986) (end 119.2911 77.6986) (width 0.8128) (layer "F.Cu") (net 9))
+  (segment (start 118.3204 100.7796) (end 118.3204 99.9204) (width 0.8128) (layer "F.Cu") (net 9))
   (segment (start 116.3 86.805) (end 116.105 87) (width 0.8128) (layer "F.Cu") (net 9))
   (segment (start 140.8811 115.7986) (end 145.9611 115.7986) (width 0.8128) (layer "F.Cu") (net 9))
