File: kicad/MegaGRRLDesktop.kicad_pcb-v0.5.kicad_pcb (KiCad board)
At the start: 2 copper layers, 124.5 x 124.5 mm, 133 parts, among them IC10 PCA9634PW, IC11 TPA6111A2DR, IC12 ESP-WROOM-32ESP-WROOM-32-NO-RF, IC14 CH340C, IC2 74HCT595N, IC3 74HCT595N, IC4 MCP23017SP, IC5 NE5532N, IC6 std:a4c6558b222b489b868198a35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, IC6A std:44d60e1deb274ae4bbd12617d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

Commit message: 2024.7.7
Parts:
- removed IC6: std:a4c6558b222b489b868198a352481a86, kicad_lceda:PWRM-TH_B0505S-3WR2
- removed IC6A: std:44d60e1deb274ae4bbd12617d1f88879, kicad_lceda:PWRM-TH_BXXXXS-1W
- removed J3: 2041021-3, MegaGRRLDesktop:SD-106M
- removed TP_5V0: , MegaGRRLDesktop:B1,27
- added 2k2: R_0603_1608Metric, Resistor_SMD:R_0603_1608Metric, F.Cu at (193.3, 141.9)
- added 4.7u: C_0603_1608Metric, Capacitor_SMD:C_0603_1608Metric, F.Cu at (209.9, 77.1)
- added REF**: std:49f2b71367e441ef98f3fd00a8fa66d5, Library:MINI560DC-DC, F.Cu at (101.5, 68.8)
- added XH2.54-9P: std:f55dec43d47241219f1ef8a3f0efb8e3, Library:CONN-TH_9P-P2.50_ZX-XH2.54-9PZZ, F.Cu at (109.2, 137.4)
- moved G*** 118.5 mm to (186.8, 153.0)
- moved G*** 28.2 mm to (100.4, 99.0)
- moved C29 11.8 mm to (120.2, 65.4)
- moved C28 6.79 mm to (121.0, 59.3)
- moved G*** 5.89 mm to (109.5, 127.0)
- moved C33 2.22 mm to (121.5, 71.5)
- renumbered REF** to SW1
Connections:
- C8 pad -: AUDIO_PSG -> AUDIO_PSG2
- R23 pad 5: Net-(R23-PadS) -> PSG_MIX1
Routing:
- net PSG_MIX1: track 0.00 -> 73.9 mm
- net Net-(R23-PadS): track 76.9 -> 5.73 mm
- net /Keys/KEY_C: track 23.1 -> 76.4 mm, vias 0 -> 1
- net /Keys/KEY_B: track 19.5 -> 64.5 mm, vias 0 -> 2
- net /Keys/KEY_DOWN: track 44.2 -> 77.0 mm
- net /Keys/KEY_A: track 25.8 -> 51.8 mm
- net /Keys/KEY_RIGHT: track 33.1 -> 49.4 mm
- net +12V: track 39.6 -> 24.5 mm
- net GND-IN: track 48.4 -> 58.7 mm
- net /Keys/KEY_UP: track 30.2 -> 39.9 mm
- net /Keys/KEY_LEFT: track 46.4 -> 53.7 mm
- net +5V: track 379.3 -> 373.3 mm
- net AUDIO_PSG2: track 0.00 -> 4.62 mm
- net AUDIO_PSG: track 11.1 -> 15.6 mm
- net +3V3: track 243.0 -> 247.2 mm
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Other:
- board text added: "2024.7.1 v0.5 1.修复0.47版本所有音频电路BUG 2.更换降压模块为效率最高，最省钱的MINI560 3.添加键盘连接器，含+5V"
- board text added: "DC 9V"
- board text added: "MegaGRRL Desktop DJ Rev.0.5 Denjhang 2024.7.1"
- board text removed: "DC 500mA"
- board text removed: "MegaGRRL Desktop DJ Rev.0.4 Denjhang 2024.6.8"
